File: Kicad/2024/PressControl.kicad_sch (KiCad schematic)
At the start: 22 parts, among them J1 Conn_01x08_Pin, J2 Conn_01x08_Socket, J5 Conn_01x08_Socket, J6 Conn_01x08_Pin, SW1 TestAlarm

Commit message: update - tested only TEST_ALARM_PIN
Connections:
- new net: Al_5Vcc?.~ (N), J?.1, K?.~
- new net: Al_5Vcc?.~ (N), J?.2, K?.~
Other:
- note removed: "Orange"
Changed lines of the file:
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@@
-    (effects (font (size 1.27 1.27)) (justify left bottom))
-  )
-  (text "Grey" (at 167.64 100.33 0)
     (effects (font (size 1.27 1.27)) (justify left bottom))
   )
@@
     (effects (font (size 1.27 1.27) (color 0 0 194 1)) (justify left bottom))
   )
-  (text "Orange\n" (at 167.64 102.87 0)
-    (effects (font (size 1.27 1.27)) (justify left bottom))
-  )
   (text "220V OUT" (at 265.43 91.44 0)
     (effects (font (size 1.27 1.27)) (justify left bottom))
@@
     (effects (font (size 1.27 1.27) (color 0 0 194 1)) (justify left bottom))
   )
-  (text "Red\n" (at 186.69 105.41 0)
+  (text "Red\n" (at 179.07 104.775 0)
     (effects (font (size 1.27 1.27)) (justify left bottom))
   )
@@
     )
   )
-  (symbol (lib_id "Graphic:SYM_Arrow_Normal") (at 189.23 93.98 0) (unit 1)
-    (in_bom yes) (on_board yes) (dnp no)
-    (property "Reference" "#SYM?" (at 189.23 92.456 0)
-      (effects (font (size 1.27 1.27)) hide)
-    )
-    (property "Value" "SYM_Arrow_Normal" (at 189.484 95.25 0)
-      (effects (font (size 1.27 1.27)) hide)
-    )
-    (property "Footprint" "" (at 189.23 93.98 0)
-      (effects (font (size 1.27 1.27)) hide)
-    )
-    (property "Datasheet" "~" (at 189.23 93.98 0)
-      (effects (font (size 1.27 1.27)) hide)
-    )
-    (property "Sim.Enable" "0" (at 189.23 93.98 0)
+  (symbol (lib_id "Graphic:SYM_Arrow_Normal") (at 193.675 95.25 0) (unit 1)
+    (in_bom yes) (on_board yes) (dnp no)
+    (property "Reference" "#SYM?" (at 193.675 93.726 0)
+      (effects (font (size 1.27 1.27)) hide)
+    )
+    (property "Value" "SYM_Arrow_Normal" (at 193.929 96.52 0)
+      (effects (font (size 1.27 1.27)) hide)
+    )
+    (property "Footprint" "" (at 193.675 95.25 0)
+      (effects (font (size 1.27 1.27)) hide)
+    )
+    (property "Datasheet" "~" (at 193.675 95.25 0)
+      (effects (font (size 1.27 1.27)) hide)
+    )
+    (property "Sim.Enable" "0" (at 193.675 95.25 0)
       (effects (font (size 1.27 1.27)) hide)
     )
@@
     )
   )
-  (symbol (lib_id "Graphic:SYM_Arrow_Normal") (at 189.23 96.52 0) (mirror y) (unit 1)
-    (in_bom yes) (on_board yes) (dnp no)
-    (property "Reference" "#SYM?" (at 189.23 94.996 0)
-      (effects (font (size 1.27 1.27)) hide)
-    )
-    (property "Value" "SYM_Arrow_Normal" (at 188.976 97.79 0)
-      (effects (font (size 1.27 1.27)) hide)
-    )
-    (property "Footprint" "" (at 189.23 96.52 0)
-      (effects (font (size 1.27 1.27)) hide)
-    )
-    (property "Datasheet" "~" (at 189.23 96.52 0)
-      (effects (font (size 1.27 1.27)) hide)
-    )
-    (property "Sim.Enable" "0" (at 189.23 96.52 0)
+  (symbol (lib_id "Graphic:SYM_Arrow_Normal") (at 194.31 97.79 0) (mirror y) (unit 1)
+    (in_bom yes) (on_board yes) (dnp no)
+    (property "Reference" "#SYM?" (at 194.31 96.266 0)
+      (effects (font (size 1.27 1.27)) hide)
+    )
+    (property "Value" "SYM_Arrow_Normal" (at 194.056 99.06 0)
+      (effects (font (size 1.27 1.27)) hide)
+    )
+    (property "Footprint" "" (at 194.31 97.79 0)
+      (effects (font (size 1.27 1.27)) hide)
+    )
+    (property "Datasheet" "~" (at 194.31 97.79 0)
+      (effects (font (size 1.27 1.27)) hide)
+    )
+    (property "Sim.Enable" "0" (at 194.31 97.79 0)
       (effects (font (size 1.27 1.27)) hide)
     )
@@
     )
   )
-  (symbol (lib_id "Graphic:SYM_Arrow_Normal") (at 189.23 99.06 0) (mirror y) (unit 1)
-    (in_bom yes) (on_board yes) (dnp no)
-    (property "Reference" "#SYM?" (at 189.23 97.536 0)
-      (effects (font (size 1.27 1.27)) hide)
-    )
-    (property "Value" "SYM_Arrow_Normal" (at 188.976 100.33 0)
-      (effects (font (size 1.27 1.27)) hide)
-    )
-    (property "Footprint" "" (at 189.23 99.06 0)
-      (effects (font (size 1.27 1.27)) hide)
-    )
-    (property "Datasheet" "~" (at 189.23 99.06 0)
-      (effects (font (size 1.27 1.27)) hide)
-    )
-    (property "Sim.Enable" "0" (at 189.23 99.06 0)
+  (symbol (lib_id "Graphic:SYM_Arrow_Normal") (at 194.945 100.33 0) (mirror y) (unit 1)
+    (in_bom yes) (on_board yes) (dnp no)
+    (property "Reference" "#SYM?" (at 194.945 98.806 0)
+      (effects (font (size 1.27 1.27)) hide)
+    )
+    (property "Value" "SYM_Arrow_Normal" (at 194.691 101.6 0)
+      (effects (font (size 1.27 1.27)) hide)
+    )
+    (property "Footprint" "" (at 194.945 100.33 0)
+      (effects (font (size 1.27 1.27)) hide)
+    )
+    (property "Datasheet" "~" (at 194.945 100.33 0)
+      (effects (font (size 1.27 1.27)) hide)
+    )
+    (property "Sim.Enable" "0" (at 194.945 100.33 0)
       (effects (font (size 1.27 1.27)) hide)
     )
@@
     )
   )
-  (symbol (lib_id "Graphic:SYM_Arrow_Normal") (at 189.23 101.6 0) (mirror y) (unit 1)
-    (in_bom yes) (on_board yes) (dnp no)
-    (property "Reference" "#SYM1" (at 189.23 100.076 0)
-      (effects (font (size 1.27 1.27)) hide)
-    )
-    (property "Value" "SYM_Arrow_Normal" (at 188.976 102.87 0)
-      (effects (font (size 1.27 1.27)) hide)
-    )
-    (property "Footprint" "" (at 189.23 101.6 0)
-      (effects (font (size 1.27 1.27)) hide)
-    )
-    (property "Datasheet" "~" (at 189.23 101.6 0)
-      (effects (font (size 1.27 1.27)) hide)
-    )
-    (property "Sim.Enable" "0" (at 189.23 101.6 0)
-      (effects (font (size 1.27 1.27)) hide)
-    )
+  (symbol (lib_id "Graphic:SYM_Arrow_Normal") (at 194.945 102.87 0) (mirror y) (unit 1)
+    (in_bom yes) (on_board yes) (dnp no)
+    (property "Reference" "#SYM1" (at 194.945 101.346 0)
+      (effects (font (size 1.27 1.27)) hide)
+    )
+    (property "Value" "SYM_Arrow_Normal" (at 194.691 104.14 0)
+      (effects (font (size 1.27 1.27)) hide)
+    )
+    (property "Footprint" "" (at 194.945 102.87 0)
+      (effects (font (size 1.27 1.27)) hide)
+    )
+    (property "Datasheet" "~" (at 194.945 102.87 0)
+      (effects (font (size 1.27 1.27)) hide)
+    )
+    (property "Sim.Enable" "0" (at 194.945 102.87 0)
+      (effects (font (size 1.27 1.27)) hide)
+    )

Commit message: update
Connections:
- net Horn: now also A?.12 (D9), J6.5 (Pin_5); no longer A?.7 (D4)
- net PumpState: now also A?.10 (D7), J6.3 (Pin_3); no longer A?.5 (D2), J6.2 (Pin_2)
- net pressControlButton: now also J6.4 (Pin_4); no longer J6.3 (Pin_3)
- net pressControlState: now also A?.9 (D6), J6.2 (Pin_2); no longer J6.4 (Pin_4)
- net at A?.11 (D8): now also R?.1
- net at A?.14 (D11): now also SW1.2
- net at A?.6 (D3): no longer R?.1
- net Elettrovalvola: no longer names the net of A?.8 (D5)
- new net: Al_5Vcc?.~ (N), J?.1, K?.~
- new net: Al_5Vcc?.~ (N), J?.2, K?.~
