File: Kicad/2024/PressControl_vanoPompe.kicad_sch (KiCad schematic)
At the start: 27 parts, among them J1 Conn_01x08_Pin, J2 Conn_01x08_Socket, J5 Conn_01x08_Socket, J6 Conn_01x08_Pin, K1 sOnOff_ClearContacts, P1 Pump, P2 Press_Control, SW1 TestAlarm, SW2 pc_Button

Commit message: update
Parts:
- removed BZ1: Passive Buzzer, symbol Device:Buzzer
- removed D1: PressControlState, symbol Device:LED
- removed D2: PumpState, symbol Device:LED
- removed J1: Conn_01x08_Pin, symbol Connector:Conn_01x08_Pin
- removed J2: Conn_01x08_Socket, symbol Connector:Conn_01x08_Socket
- removed R? (x2): 470, symbol Device:R
- removed RL1: Relay_5V_LL, symbol lnDevice:Relay_5V_LL
- removed SW?: PCButton, symbol LnDevice:PulsanteNO
- added J1: Conn_01x08_Socket, symbol Connector:Conn_01x08_Socket
- added J2: Conn_01x08_Pin, symbol Connector:Conn_01x08_Pin
- added RL2: Relay_LowLevel, symbol lnDevice:Relay_LowLevel
- Al_5Vcc?: footprint 5V pressControl -> 5Vcc
- SW2: value pc_Button -> startPControl
Connections:
- net GND: now also J2.8 (Pin_8), RL2.~
- net VCC: now also J2.1 (Pin_1)
- net at K?.8, P2.~ (2): now also K1. (c), RL2.~; no longer Al_5Vcc?.~ (N), J?.1
- net at SW1.2: no longer A1.15 (D12)
- net at A1.14 (D11): no longer SW2.2
- new net: Al_5Vcc?.~ (N), J?.1, K1. (c), K?.9, P2.~ (2)
- new net: Al_5Vcc?.~ (N), J?.2, K1. (c), RL2.~
- new net: K?.8, P1.~ (2), P2.~ (2)
- new net arduino_PControl: J1.3 (Pin_3)
- new net sonoff_PControl: J1.2 (Pin_2)
Other:
- note removed: "Active Buzzer"
- note removed: "Active Buzzer è messo come emergenza nel caso si dovesse rimuovere Arduino. Suona in modo continuo quando la pompa è accesa. Il jumper si trova dietro il frutto."
- note removed: "Frutto del PressControl nel Quadro elettrico del Salone"
- note removed: "Il filo Arancio porta i 5Volt provenienti dalla cisterna. L'ho messo in questo modo per rendere indipendente il frutto del press control dala presenza di Arduino."
- note removed: "Passive Buzzer"
- note removed: "Shield"
- note removed: "da collegare"
- moved on the sheet: A1, D3

Commit message: update
Parts:
- removed J1, J5: Conn_01x08_Socket, symbol Connector:Conn_01x08_Socket
- removed J2, J6: Conn_01x08_Pin, symbol Connector:Conn_01x08_Pin
- removed RL2: Relay_LowLevel, symbol lnDevice:Relay_LowLevel
- added BZ1: Buzzer Active, symbol lnDevice:Buzzer Active
- added BZ2: Buzzer, symbol lnDevice:Buzzer Passive
- added D1: PressControlState, symbol Device:LED
- added D2: PumpLed, symbol Device:LED
- added D4: DIODE, symbol lnDiodiTransistors:DIODE
- added J1: SIP_05, symbol lnConnectors:SIP_05
- added J2, J5, J6: SIP_05, symbol lnConnectors:SIP_03
- added J3: Conn_01x08_Pin, symbol Connector:Conn_01x08_Pin
- added J4: SIP_05, symbol lnConnectors:SIP_04
- added J7: SIP_04, symbol lnConnectors:SIP_04
- added K2: Relayx1_Module, symbol lnDevice:Relayx1_Module
- added MM1, MM2: Mammuth_02a, symbol lnConnectors:Mammuth_02a
- added R1, R2: 470, symbol Device:R
- added SW3: startPControl, symbol LnDevice:PulsanteNO
- K1: renamed from K?; footprint (none) -> PC_relay
- K?: footprint (none) -> Pump_relay
- R?: value 1K -> 10K
- SW2: value startPControl -> start_PControl
Connections:
- net +5V: now also K2.1 (VCC)
- net GND: now also SW1.1, SW2.1, K2.2 (GND)
- net PumpState: now also A1.11 (D8)
- net arduino_PControl: now also K2.3 (IN1)
- net pressControlState: now also A1.12 (D9)
- net sonoff_PControl: now also A1.14 (D11), K1.~, R?.2, SW2.2
- net sonoff_emergency: now reaches R?.1
- net sonoff_emergency: now also A1.13 (D10)
- net at SW1.2: now also A1.15 (D12)
- new net: J4.1, J?.1, P2.~ (2)
- new net: J7.1, J?.2
- new net: Al_5Vcc?.~ (N), J4.2
- new net: Al_5Vcc?.~ (N), J7.2
- new net: J2.1, K1. (c), K2.3 (IN1)
- new net: J2.2, P2.~ (2)
- new net: J2.3, K1.8
- new net: J5.2, K?.8
- new net: J6.2, K?.9
- new net: J4.4, K1.9
- new net: D1.2 (A), R1.1
- new net: R1.2, R2.2
- new net: J6.1, P2.~ (2)
- new net: J6.3, P1.~ (2)
- new net: J5.1, P2.~ (2)
- new net: J5.3, P1.~ (2)
- new net: J4.3, K1. (c)
- new net: D2.2 (A), R2.1
- new net: J7.3, K1. (c)
- new net: J7.4, K1. (c), K2.2 (GND)
Other:
- note added: "Frutto del PressControl nel Quadro elettrico del Salone"
- note added: "Il filo Arancio porta i 5Volt provenienti dalla cisterna. L'ho messo in questo modo per rendere indipendente il frutto del press control dala presenza di Arduino."
- note added: "Shield"
- note removed: "220V IN"
- note removed: "Black"
- note removed: "Bleu"
- note removed: "Brown"
- note removed: "Green"
- moved on the sheet: D3, K1

Commit message: creata funzione per short/long press button
Connections:
- net sonoff_PControl: now also D4.2 (K); no longer K1.~
- net at D4.1 (A): now also K1.~
- new net: J2.1, K1. (c), K2.3 (IN1)
Changed lines of the file:
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@@
 	(wire
 		(pts
-			(xy 92.71 82.55) (xy 92.71 78.74)
+			(xy 95.25 82.55) (xy 95.25 80.01)
 		)
 		(stroke
@@
 	(wire
 		(pts
-			(xy 120.65 73.66) (xy 119.38 73.66)
+			(xy 120.65 73.66) (xy 116.84 73.66)
 		)
 		(stroke
@@
 	(wire
 		(pts
-			(xy 101.6 82.55) (xy 92.71 82.55)
+			(xy 95.25 82.55) (xy 101.6 82.55)
 		)
 		(stroke
@@
 			(type default)
 			(color 132 0 0 1)
+		)
+	)
+	(wire
+		(pts
+			(xy 109.22 73.66) (xy 86.36 73.66)
+		)
+		(stroke
+			(width 0)
+			(type default)
 		)
 	)
@@
 	(global_label "sonoff_PControl"
 		(shape input)
-		(at 119.38 73.66 180)
+		(at 86.36 73.66 180)
 		(fields_autoplaced yes)
 		(effects
@@
 		)
 		(property "Intersheetrefs" "${INTERSHEET_REFS}"
-			(at 104.9453 73.66 0)
+			(at 71.9253 73.66 0)
 			(effects
 				(font
@@
 	(symbol
 		(lib_id "power:+5V")
-		(at 92.71 78.74 0)
+		(at 95.25 80.01 0)
 		(unit 1)
 		(exclude_from_sim no)
@@
 		(fields_autoplaced yes)
 		(property "Reference" "#PWR03"
-			(at 92.71 82.55 0)
+			(at 95.25 83.82 0)
 			(effects
 				(font
@@
 		)
 		(property "Value" "+5V"
-			(at 92.71 73.66 0)
+			(at 95.25 74.93 0)
 			(effects
 				(font
@@
 		)
 		(property "Footprint" ""
-			(at 92.71 78.74 0)
+			(at 95.25 80.01 0)
 			(effects
 				(font
@@
 		)
 		(property "Datasheet" ""
-			(at 92.71 78.74 0)
+			(at 95.25 80.01 0)
 			(effects
 				(font
@@
 		)
 		(property "Description" "Power symbol creates a global label with name \"+5V\""
-			(at 92.71 78.74 0)
+			(at 95.25 80.01 0)
 			(effects
 				(font
@@
 	(symbol
 		(lib_id "lnDiodiTransistors:DIODE")
-		(at 232.41 125.73 0)
-		(unit 1)
-		(exclude_from_sim no)
-		(in_bom yes)
-		(on_board yes)
-		(dnp no)
-		(fields_autoplaced yes)
+		(at 113.03 73.66 0)
+		(mirror y)
+		(unit 1)
+		(exclude_from_sim no)
+		(in_bom yes)
+		(on_board yes)
+		(dnp no)
 		(property "Reference" "D4"
-			(at 232.4481 121.92 0)
+			(at 112.9919 69.85 0)
 			(effects
 				(font
@@
 		)
 		(property "Value" "DIODE"
-			(at 232.4481 121.92 0)
+			(at 112.9919 69.85 0)
 			(effects
 				(font
@@
 		)
 		(property "Footprint" ""
-			(at 232.41 125.73 0)
+			(at 113.03 73.66 0)
 			(effects
 				(font
@@
 		)
 		(property "Datasheet" ""
-			(at 232.41 125.73 0)
+			(at 113.03 73.66 0)
 			(effects
 				(font
@@
 		)
 		(property "Description" ""
-			(at 232.41 125.73 0)
-			(effects
-				(font
+			(at 113.03 73.66 0)
+			(effects
+				(font
