File: Kicad/2024/PressControl_con_Alim.kicad_sch (KiCad schematic)
At the start: 51 parts, among them J1 SIP_05, J10 Conn_01x08_Socket, J11 SIP_01, J12 SIP_01, J13 SIP_01, J2 SIP_05, J3 Conn_01x08_Pin, J4 SIP_05, J5 SIP_05, J6 SIP_05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

Commit message: kicad schematic changes
Connections:
- net at Al_5Vcc2.~ (-), P1.~ (2), P2.~ (1): now also J13.1; no longer J12.1
- new net: Al_5Vcc1.~ (-), Al_5Vcc?.~ (-), J9.1, J?.1, K1. (c), P2.~ (1)
- new net: Al_5Vcc?.~ (-), J8.1, J?.2, K1. (c), K2.3
- new net: Al_5Vcc1.~ (-), J11.1, K1. (c), K2.2, P2.~ (1)
- new net: Al_5Vcc2.~ (-), J12.1, P1.~ (2), P2.~ (1)
