File: Kicad/2025/PressControl_ESP32_2relay.kicad_sch (KiCad schematic)
At the start: 34 parts, among them J10 Conn_01x08_Socket, J11 Conn_01x08_Socket, J12 SIP_01, J13 SIP_01, J14 Conn_01x08_Pin, J15 Conn_01x08_Socket, J16 Conn_01x08_Pin, J3 Conn_01x08_Pin, J8 Conn_01x08_Socket, J9 Conn_01x08_Pin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

Commit message: ''
Connections:
- net activeBuzzer: now also U1.37 (G.23); no longer U1.15 (G.13)
- net passiveBuzzer: now also U1.36 (G.22); no longer U1.13 (G.12)
- net pressControlLed: now also U1.9 (G.25); no longer U1.12 (G.14)
- net pumpLED: now also U1.10 (G.26); no longer U1.23 (G.15)
- net at K3.3 (IN1): now also U1.28 (G.17)
- new net: K1.9, K3.2 (GND), P2.~ (2)
- now unconnected: K3.2 (GND)

Commit message: 'sembra la versione base funzionante. Ho dovuto mettere SSHCLIENT=false'
Parts:
- D1, D4: value PressControlLed -> pressControlLED
- D2, D5: value PumpLed -> PumpLED
Connections:
- net at K3.3 (IN1): now also U1.28 (G.17)
- net pressControlLed renamed pressControlLED
- new net: K1.9, K3.2 (GND), P2.~ (2)
- now unconnected: K3.2 (GND)
Changed lines of the file:
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@@
 		)
 	)
-	(label "pressControlLed"
+	(label "pressControlLED"
 		(at 201.93 90.17 0)
 		(effects
@@
 			)
 		)
-		(property "Value" "PressControlLed"
+		(property "Value" "pressControlLED"
 			(at 24.13 136.525 0)
 			(effects
@@
 			)
 		)
-		(property "Value" "PumpLed"
+		(property "Value" "PumpLED"
 			(at 35.56 77.216 0)
 			(effects
@@
 			)
 		)
-		(property "Value" "PumpLed"
+		(property "Value" "PumpLED"
 			(at 35.56 143.256 0)
 			(effects
@@
 			)
 		)
-		(property "Value" "PressControlLed"
+		(property "Value" "pressControlLED"
 			(at 25.4 71.12 0)
 			(effects

Commit message: first released version
Parts:
- removed U2: ESP32-WROOM-32e con 2 relays, RF_Module:ESP32-WROOM-32, symbol ln_IC:ESP32-WROOM-32-2relays
- added J1: Conn_01x08_Pin, symbol Connector:Conn_01x04_Pin
- added J2: Conn_01x08_Socket, symbol Connector:Conn_01x04_Socket
Connections:
- net GND: now also J2.2 (Pin_2), J2.3 (Pin_3); no longer K1.1 (T1), K2.1 (T1)
- net PressControlState: now also J2.4 (Pin_4)
- net PumpState: now also J2.1 (Pin_1); no longer K2.5 (C1)
- net pressControlState: no longer K1.5 (C1)
- net at K3.3 (IN1): now also U1.28 (G.17)
- new net: J1.4 (Pin_4), K1.1 (T1)
- new net: J1.3 (Pin_3), K1.5 (C1)
- new net: K1.9, K3.2 (GND), P2.~ (2)
- new net: J1.1 (Pin_1), K2.5 (C1)
- new net: J1.2 (Pin_2), K2.1 (T1)
- now unconnected: K3.2 (GND)

Commit message: update kicad
Parts:
- added CB3: CircuitBreaker_1+1P, symbol lnConnectors:CircuitBreaker_1+1P
Connections:
- net at J?.2, K3.3 (IN1): now also K3.2 (GND)
- net at K3.1 (VCC): now also CB3.1
- net at K3.3 (IN1): now also U1.28 (G.17)
- new net: CB3.3, J?.1
- new net: CB3.3, K1.8, P2.~ (2)
- new net: CB3.2, K1.9, K3.2 (GND), P2.~ (2)
- now unconnected: K3.2 (GND)
Other:
- note added: "Il secondo relè, quando OFF, porta tensione al CB. Il secondo relè viene acceso, in caso di Allarme, per toglere tensione al pressControl e quindi alla pompa nel caso che spegnendo il primo relè l'allarme non cessasse."

Commit message: kicad schematic changes
Connections:
- net at K3.1: now also CB3.1
- net at K3.3: now also U1.28 (G.17)
- new net: J?.2, K3.2, K3.3
- now unconnected: K3.2 (GND)
